Commit message: Run each AMR under its own namespace; start one to three of them
The Gazebo topics, bridge, robot_state_publisher, Nav2, tag reader and task executor
of a robot now all live under /amr_N, with the robot's own TF tree on /amr_N/tf, so
several robots can share one world.

- amr_description: namespace:= xacro argument for the Gazebo topics
- amr_gazebo: sim.launch.py is the world and /clock only; robot.launch.py adds one
  robot with its own bridge (expand_gz_topic_names)
- amr_navigation: navigation.launch.py starts one robot's Nav2 (AMCL at its start
  pose) and tag reader; it replaces bringup.launch.py
- amr_bringup: sim.launch.py starts Gazebo, 1 to 3 robots parked in q1 to q3 and
  RViz; fleet.launch.py takes the same robots:=
- amr_task_executor: relative dock_robot and cmd_vel names

File: amr_description/urdf/amr.gazebo.xacro (robot description, xacro)
@@ -29,7 +29,7 @@
       <max_angular_velocity>1.5</max_angular_velocity>
       <max_linear_acceleration>0.5</max_linear_acceleration>
-      <topic>cmd_vel</topic>
-      <odom_topic>odom</odom_topic>
-      <tf_topic>tf</tf_topic>
+      <topic>/${ns}/cmd_vel</topic>
+      <odom_topic>/${ns}/odom</odom_topic>
+      <tf_topic>/${ns}/tf</tf_topic>
       <frame_id>odom</frame_id>
       <child_frame_id>base_footprint</child_frame_id>
@@ -41,5 +41,5 @@
     <plugin filename="gz-sim-joint-state-publisher-system"
             name="gz::sim::systems::JointStatePublisher">
-      <topic>joint_states</topic>
+      <topic>/${ns}/joint_states</topic>
     </plugin>
   </gazebo>
@@ -47,5 +47,5 @@
   <gazebo reference="lidar_link">
     <sensor name="lidar" type="gpu_lidar">
-      <topic>scan</topic>
+      <topic>/${ns}/scan</topic>
       <gz_frame_id>lidar_link</gz_frame_id>
       <update_rate>10</update_rate>

File: amr_description/urdf/amr.urdf.xacro (robot description, xacro)
@@ -8,4 +8,8 @@
   -->
   <xacro:property name="mesh_dir" value="file://$(find amr_description)/meshes/mir"/>
+  <!-- The robot's name. Its Gazebo topics are /<namespace>/cmd_vel, /<namespace>/scan, ...
+       so several AMRs can share one world: xacro amr.urdf.xacro namespace:=amr_2 -->
+  <xacro:arg name="namespace" default="amr_1"/>
+  <xacro:property name="ns" value="$(arg namespace)"/>
   <!-- ========== Dimensions (metres, kg), measured from the MiR100 meshes ========== -->
   <xacro:property name="base_mass" value="58.0"/>
@@ -244,5 +248,5 @@
   <gazebo reference="camera_link">
     <sensor name="floor_camera" type="camera">
-      <topic>camera/image</topic>
+      <topic>/${ns}/camera/image</topic>
       <gz_frame_id>camera_optical_link</gz_frame_id>
       <update_rate>15</update_rate>
